File: TA8-FDC.kicad_sch (KiCad schematic)
At the start: 69 parts, among them IC101 SED9420C, IC102 LS74, IC103 LS32, IC104 74LS95, IC105 LS10, IC106 LS139, IC107 74LS641, IC108 LS368, IC109 LS08, IC110 LS02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

Commit message: Add files via upload
corrected a couple of error on schematics
Parts:
- removed D101: IS2473, Diode_THT:D_A-405_P10.16mm_Horizontal, symbol Device:D
- removed IC3: FDC9266, Package_DIP:DIP-40_W15.24mm_Socket, symbol 8Bit_Parts:FDC9266
- added D1: IS2473, Diode_THT:D_A-405_P10.16mm_Horizontal, symbol Device:D
Connections:
- net at IC110.8: now also IC112.3; no longer IC108.3
- net toIORQ: now reaches IC105.5, IC118.10
- net toIORQ: now also IC112.2
- net at R102.2: now also D1.1 (K); no longer C102.2
- net at R106.2: now also C102.2, D1.2 (A)
- net at IC112.1: now also IC108.3
- no-connect marks 55 -> 49
Other:
- note removed: "FDC"
- moved on the sheet: IC108A, IC108D, IC110C, IC112A

Commit message: Fixed C117
Parts:
- removed C117: 10µF, Capacitor_THT:CP_Axial_L10.0mm_D4.5mm_P15.00mm_Horizontal, symbol Device:C
- added C117: 10uF, Capacitor_THT:CP_Axial_L10.0mm_D4.5mm_P15.00mm_Horizontal, symbol Device:C_Polarized
Connections:
- net +5V: now also C117.1
- net GND: now also C117.2
Changed lines of the file:
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@@
   (junction (at 140.97 237.49) (diameter 0) (color 0 0 0 0)
   )
+  (junction (at 156.21 237.49) (diameter 0) (color 0 0 0 0)
+  )
   (junction (at 290.83 118.11) (diameter 0) (color 0 0 0 0)
   )
@@
   (junction (at 274.32 97.79) (diameter 0) (color 0 0 0 0)
   )
-  (junction (at 156.21 237.49) (diameter 0) (color 0 0 0 0)
-  )
   (junction (at 80.01 245.11) (diameter 0) (color 0 0 0 0)
   )
@@
     (stroke (width 0) (type default))
   )
-  (wire (pts (xy 156.21 237.49) (xy 161.29 237.49))
+  (wire (pts (xy 146.05 237.49) (xy 156.21 237.49))
     (stroke (width 0) (type default))
   )
@@
     (stroke (width 0) (type default))
   )
-  (wire (pts (xy 146.05 237.49) (xy 156.21 237.49))
-    (stroke (width 0) (type default))
-  )
   (wire (pts (xy 229.87 229.87) (xy 243.84 229.87))
     (stroke (width 0) (type default))
@@
     (stroke (width 0) (type default))
   )
+  (wire (pts (xy 156.21 237.49) (xy 161.29 237.49))
+    (stroke (width 0) (type default))
+  )
   (wire (pts (xy 256.54 234.95) (xy 256.54 259.08))
     (stroke (width 0) (type default))
@@
     )
   )
-  (symbol (lib_id "Device:C") (at 156.21 241.3 180) (unit 1)
-    (in_bom yes) (on_board yes) (dnp no)
-    (property "Reference" "C117" (at 156.21 234.95 0)
-      (effects (font (size 1.27 1.27)))
-    )
-    (property "Value" "10µF" (at 160.02 238.76 0)
-      (effects (font (size 1.27 1.27)))
-    )
-    (property "Footprint" "Capacitor_THT:CP_Axial_L10.0mm_D4.5mm_P15.00mm_Horizontal" (at 155.2448 237.49 0)
-      (effects (font (size 1.27 1.27)) hide)
-    )
-    (property "Datasheet" "~" (at 156.21 241.3 0)
-      (effects (font (size 1.27 1.27)) hide)
-    )
-    (pin "1")
-    (pin "2")
-    (instances
-      (project "TA8-FDC"
-        (path "/850a6d6d-37bd-4b54-9e36-0aa92a95f89b"
-          (reference "C117") (unit 1)
-        )
-      )
-    )
-  )
   (symbol (lib_id "Connector:Barrel_Jack") (at 372.11 39.37 0) (unit 1)
     (in_bom yes) (on_board yes) (dnp no) (fields_autoplaced)
@@
         )
       )
+    )
+  )
+  (symbol (lib_id "Device:C_Polarized") (at 156.21 241.3 0) (unit 1)
+    (in_bom yes) (on_board yes) (dnp no) (fields_autoplaced)
+    (property "Reference" "C117" (at 159.131 239.1989 0)
+      (effects (font (size 1.27 1.27)) (justify left))
+    )
+    (property "Value" "10uF" (at 159.131 241.6231 0)
+      (effects (font (size 1.27 1.27)) (justify left))
+    )
+    (property "Footprint" "Capacitor_THT:CP_Axial_L10.0mm_D4.5mm_P15.00mm_Horizontal" (at 157.1752 245.11 0)
+      (effects (font (size 1.27 1.27)) hide)
+    )
+    (property "Datasheet" "~" (at 156.21 241.3 0)
+      (effects (font (size 1.27 1.27)) hide)
+    )
+    (pin "1")
+    (pin "2")
+    (instances
+      (project "TA8-FDC"
+        (path "/850a6d6d-37bd-4b54-9e36-0aa92a95f89b"
+          (reference "C117") (unit 1)
+        )
+      )
